File: TH-XWhatsIt/TH-XWhatsIt.sch (KiCad schematic (older format))
At the start: 25 parts, among them J1 BEAMSPRING CONNECTOR, J3 EXPANSION HEADER, U1 MCP4921-EP, U2 LM339, U3 74HCT595, U4 74HCT595, U5 ProMicro, U7 74HCT595

Commit message: added lcsc numbers for remaining chips, changed some silkscreen to match parts, removed stay-upright flag from all silkscreen, etc...
Parts:
- U1: value MCP4921-EP -> MCP4921-E
- U2: value LM339 -> LM339A; LCSC (none) -> C74559
- U3, U4, U7: value 74HCT595 -> 74AHC595; LCSC (none) -> C5520
Changed lines of the file:
@@
 P 2100 7250
 F 0 "U2" H 2058 7296 50  0000 L CNN
-F 1 "LM339" H 2058 7205 50  0000 L CNN
+F 1 "LM339A" H 2058 7205 50  0000 L CNN
 F 2 "Package_SO:SOIC-14_3.9x8.7mm_P1.27mm" H 2050 7350 50  0001 C CNN
 F 3 "http://www.ti.com/lit/ds/symlink/lm339.pdf" H 2150 7450 50  0001 C CNN
+F 4 "C74559" H 2100 7250 50  0001 C CNN "LCSC"
 	5    2100 7250
 	1    0    0    -1
@@
 P 5275 1575
 F 0 "U3" H 5275 2356 50  0000 C CNN
-F 1 "74HCT595" H 5275 2265 50  0000 C CNN
+F 1 "74AHC595" H 5275 2265 50  0000 C CNN
 F 2 "Package_SO:SOIC-16_3.9x9.9mm_P1.27mm" H 5275 1575 50  0001 C CNN
 F 3 "https://assets.nexperia.com/documents/data-sheet/74HC_HCT595.pdf" H 5275 1575 50  0001 C CNN
+F 4 "C5520" H 5275 1575 50  0001 C CNN "LCSC"
 	1    5275 1575
 	1    0    0    -1
@@
 P 5275 3350
 F 0 "U4" H 5275 4131 50  0000 C CNN
-F 1 "74HCT595" H 5275 4040 50  0000 C CNN
+F 1 "74AHC595" H 5275 4040 50  0000 C CNN
 F 2 "Package_SO:SOIC-16_3.9x9.9mm_P1.27mm" H 5275 3350 50  0001 C CNN
 F 3 "https://assets.nexperia.com/documents/data-sheet/74HC_HCT595.pdf" H 5275 3350 50  0001 C CNN
+F 4 "C5520" H 5275 3350 50  0001 C CNN "LCSC"
 	1    5275 3350
 	1    0    0    -1
@@
 P 5275 5125
 F 0 "U7" H 5275 5906 50  0000 C CNN
-F 1 "74HCT595" H 5275 5815 50  0000 C CNN
+F 1 "74AHC595" H 5275 5815 50  0000 C CNN
 F 2 "Package_SO:SOIC-16_3.9x9.9mm_P1.27mm" H 5275 5125 50  0001 C CNN
 F 3 "https://assets.nexperia.com/documents/data-sheet/74HC_HCT595.pdf" H 5275 5125 50  0001 C CNN
+F 4 "C5520" H 5275 5125 50  0001 C CNN "LCSC"
 	1    5275 5125
 	1    0    0    -1
@@
 P 2300 1575
 F 0 "U2" H 2300 1942 50  0000 C CNN
-F 1 "LM339" H 2300 1851 50  0000 C CNN
+F 1 "LM339A" H 2300 1851 50  0000 C CNN
 F 2 "Package_SO:SOIC-14_3.9x8.7mm_P1.27mm" H 2250 1675 50  0001 C CNN
 F 3 "http://www.ti.com/lit/ds/symlink/lm339.pdf" H 2350 1775 50  0001 C CNN
+F 4 "C74559" H 2300 1575 50  0001 C CNN "LCSC"
 	1    2300 1575
 	1    0    0    -1
@@
 P 2300 2175
 F 0 "U2" H 2300 2542 50  0000 C CNN
-F 1 "LM339" H 2300 2451 50  0000 C CNN
+F 1 "LM339A" H 2300 2451 50  0000 C CNN
 F 2 "Package_SO:SOIC-14_3.9x8.7mm_P1.27mm" H 2250 2275 50  0001 C CNN
 F 3 "http://www.ti.com/lit/ds/symlink/lm339.pdf" H 2350 2375 50  0001 C CNN
+F 4 "C74559" H 2300 2175 50  0001 C CNN "LCSC"
 	2    2300 2175
 	1    0    0    -1
@@
 P 2300 2775
 F 0 "U2" H 2300 3142 50  0000 C CNN
-F 1 "LM339" H 2300 3051 50  0000 C CNN
+F 1 "LM339A" H 2300 3051 50  0000 C CNN
 F 2 "Package_SO:SOIC-14_3.9x8.7mm_P1.27mm" H 2250 2875 50  0001 C CNN
 F 3 "http://www.ti.com/lit/ds/symlink/lm339.pdf" H 2350 2975 50  0001 C CNN
+F 4 "C74559" H 2300 2775 50  0001 C CNN "LCSC"
 	3    2300 2775
 	1    0    0    -1
@@
 P 2300 3375
 F 0 "U2" H 2300 3742 50  0000 C CNN
-F 1 "LM339" H 2300 3651 50  0000 C CNN
+F 1 "LM339A" H 2300 3651 50  0000 C CNN
 F 2 "Package_SO:SOIC-14_3.9x8.7mm_P1.27mm" H 2250 3475 50  0001 C CNN
 F 3 "http://www.ti.com/lit/ds/symlink/lm339.pdf" H 2350 3575 50  0001 C CNN
+F 4 "C74559" H 2300 3375 50  0001 C CNN "LCSC"
 	4    2300 3375
 	1    0    0    -1
@@
 P 9075 1400
 F 0 "U1" H 9719 1446 50  0000 L CNN
-F 1 "MCP4921-EP" H 9525 1350 50  0000 L CNN
+F 1 "MCP4921-E" H 9525 1350 50  0000 L CNN
 F 2 "Package_SO:SOIC-8_3.9x4.9mm_P1.27mm" H 9075 1400 50  0001 C CIN
 F 3 "http://ww1.microchip.com/downloads/en/devicedoc/21897a.pdf" H 9075 1400 50  0001 C CNN
