File: CompactBeamspring/CompactBeamspring.sch (KiCad schematic (older format))
At the start: 32 parts, among them J1 BEAMSPRING CONNECTOR, J2 PadsToShort, J3 EXPANSION HEADER, U1 MCP4921-E, U2 LM339A, U3 74AHC595, U4 74AHC595, U5 ProMicro, U7 74AHC595

Commit message: Fixup wrong footprint reference
Parts:
- J1: footprint TH-XWhatsIt:30-pin-universal-beamspring-connector_v2 -> TH-XWhatsIt:30-pin-universal-beamspring-connector_v3_onlyflat
Changed lines of the file:
@@
 F 0 "J1" H 2955 5267 50  0000 L CNN
 F 1 "BEAMSPRING CONNECTOR" H 2955 5176 50  0000 L CNN
-F 2 "TH-XWhatsIt:30-pin-universal-beamspring-connector_v2" H 2875 5275 50  0001 C CNN
+F 2 "TH-XWhatsIt:30-pin-universal-beamspring-connector_v3_onlyflat" H 2875 5275 50  0001 C CNN
 F 3 "~" H 2875 5275 50  0001 C CNN
 	1    2875 5275

Commit message: Updated 100k resistor LCSC part numbers
Parts:
- R10, R11, R12, R9: LCSC C17407 -> C149504
Changed lines of the file:
@@
 F 2 "Resistor_SMD:R_0805_2012Metric_Pad1.15x1.40mm_HandSolder" V 1380 1325 50  0001 C CNN
 F 3 "~" H 1450 1325 50  0001 C CNN
-F 4 "C17407" H 1450 1325 50  0001 C CNN "LCSC"
+F 4 "C149504" H 1450 1325 50  0001 C CNN "LCSC"
 	1    1450 1325
 	1    0    0    -1
@@
 F 2 "Resistor_SMD:R_0805_2012Metric_Pad1.15x1.40mm_HandSolder" V 1380 1925 50  0001 C CNN
 F 3 "~" H 1450 1925 50  0001 C CNN
-F 4 "C17407" H 1450 1925 50  0001 C CNN "LCSC"
+F 4 "C149504" H 1450 1925 50  0001 C CNN "LCSC"
 	1    1450 1925
 	1    0    0    -1
@@
 F 2 "Resistor_SMD:R_0805_2012Metric_Pad1.15x1.40mm_HandSolder" V 1380 2525 50  0001 C CNN
 F 3 "~" H 1450 2525 50  0001 C CNN
-F 4 "C17407" H 1450 2525 50  0001 C CNN "LCSC"
+F 4 "C149504" H 1450 2525 50  0001 C CNN "LCSC"
 	1    1450 2525
 	1    0    0    -1
@@
 F 2 "Resistor_SMD:R_0805_2012Metric_Pad1.15x1.40mm_HandSolder" V 1380 3125 50  0001 C CNN
 F 3 "~" H 1450 3125 50  0001 C CNN
-F 4 "C17407" H 1450 3125 50  0001 C CNN "LCSC"
+F 4 "C149504" H 1450 3125 50  0001 C CNN "LCSC"
 	1    1450 3125
 	1    0    0    -1

Commit message: Updated shift register LCSC part number
Parts:
- U3, U4, U7: LCSC C5520 -> C2682116
Changed lines of the file:
@@
 F 2 "Package_SO:SOIC-16_3.9x9.9mm_P1.27mm" H 5275 1575 50  0001 C CNN
 F 3 "https://assets.nexperia.com/documents/data-sheet/74HC_HCT595.pdf" H 5275 1575 50  0001 C CNN
-F 4 "C5520" H 5275 1575 50  0001 C CNN "LCSC"
+F 4 "C2682116" H 5275 1575 50  0001 C CNN "LCSC"
 	1    5275 1575
 	1    0    0    -1
@@
 F 2 "Package_SO:SOIC-16_3.9x9.9mm_P1.27mm" H 5275 3350 50  0001 C CNN
 F 3 "https://assets.nexperia.com/documents/data-sheet/74HC_HCT595.pdf" H 5275 3350 50  0001 C CNN
-F 4 "C5520" H 5275 3350 50  0001 C CNN "LCSC"
+F 4 "C2682116" H 5275 3350 50  0001 C CNN "LCSC"
 	1    5275 3350
 	1    0    0    -1
@@
 F 2 "Package_SO:SOIC-16_3.9x9.9mm_P1.27mm" H 5275 5125 50  0001 C CNN
 F 3 "https://assets.nexperia.com/documents/data-sheet/74HC_HCT595.pdf" H 5275 5125 50  0001 C CNN
-F 4 "C5520" H 5275 5125 50  0001 C CNN "LCSC"
+F 4 "C2682116" H 5275 5125 50  0001 C CNN "LCSC"
 	1    5275 5125
 	1    0    0    -1

Commit message: Revert "Updated shift register LCSC part number"
This reverts commit 109b71d9faab148fe864110445be2db0dc0f59e0.
Parts:
- U3, U4, U7: LCSC C2682116 -> C5520
Changed lines of the file:
@@
 F 2 "Package_SO:SOIC-16_3.9x9.9mm_P1.27mm" H 5275 1575 50  0001 C CNN
 F 3 "https://assets.nexperia.com/documents/data-sheet/74HC_HCT595.pdf" H 5275 1575 50  0001 C CNN
-F 4 "C2682116" H 5275 1575 50  0001 C CNN "LCSC"
+F 4 "C5520" H 5275 1575 50  0001 C CNN "LCSC"
 	1    5275 1575
 	1    0    0    -1
@@
 F 2 "Package_SO:SOIC-16_3.9x9.9mm_P1.27mm" H 5275 3350 50  0001 C CNN
 F 3 "https://assets.nexperia.com/documents/data-sheet/74HC_HCT595.pdf" H 5275 3350 50  0001 C CNN
-F 4 "C2682116" H 5275 3350 50  0001 C CNN "LCSC"
+F 4 "C5520" H 5275 3350 50  0001 C CNN "LCSC"
 	1    5275 3350
 	1    0    0    -1
@@
 F 2 "Package_SO:SOIC-16_3.9x9.9mm_P1.27mm" H 5275 5125 50  0001 C CNN
 F 3 "https://assets.nexperia.com/documents/data-sheet/74HC_HCT595.pdf" H 5275 5125 50  0001 C CNN
-F 4 "C2682116" H 5275 5125 50  0001 C CNN "LCSC"
+F 4 "C5520" H 5275 5125 50  0001 C CNN "LCSC"
 	1    5275 5125
 	1    0    0    -1
